File: Board/_DRM_Watch_v3/DRM_Watch_V3.kicad_sch (KiCad schematic)
At the start: 103 parts, among them J1 TYPE-C-31-M-12, J2 687110149022, Q1 2N7002LT1G, U3 TP4056, U4 DS3231S, Y1 3225 4PIN 40Mhz 3.2*2.5mm Pas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

Commit message: doc
Parts:
- C16: Model (none) -> Capacitor SMD 1206 10NF X7R 200V
- J2: value 687110149022 -> FPC 10pin 0.5mm pitch; Link (none) -> https://www.aliexpress.us/item/10000348360254.html; now in the parts list
- gave numbers to parts that had none: 2
Changed lines of the file:
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@@
   (symbol (lib_id "Project-Lib:ESP32-S2") (at 179.07 110.49 0) (unit 1)
     (in_bom yes) (on_board yes) (dnp no) (fields_autoplaced)
-    (property "Reference" "U?" (at 181.2641 153.67 0)
+    (property "Reference" "U1" (at 181.2641 153.67 0)
       (effects (font (size 1.27 1.27)) (justify left) hide)
     )
@@
       (project "DRM_Watch_V3"
         (path "/d50c768c-843d-4a19-b0bf-8bd21b6b9231"
-          (reference "U?") (unit 1)
+          (reference "U1") (unit 1)
         )
       )
@@
       (effects (font (size 1.27 1.27)) hide)
     )
+    (property "Model" "Capacitor SMD 1206 10NF X7R 200V" (at 281.94 254 0)
+      (effects (font (size 1.27 1.27)) hide)
+    )
     (pin "2")
     (pin "1")
@@
   (symbol (lib_id "Project-Lib:HV857") (at 255.27 236.22 0) (unit 1)
     (in_bom yes) (on_board yes) (dnp no)
-    (property "Reference" "U?" (at 255.27 248.92 0)
+    (property "Reference" "U5" (at 255.27 248.92 0)
       (effects (font (size 1.27 1.27)) hide)
     )
@@
       (project "DRM_Watch_V3"
         (path "/d50c768c-843d-4a19-b0bf-8bd21b6b9231"
-          (reference "U?") (unit 1)
+          (reference "U5") (unit 1)
         )
       )
@@
   )
   (symbol (lib_id "Project-Lib:687110149022") (at 368.3 205.74 0) (mirror x) (unit 1)
-    (in_bom no) (on_board yes) (dnp no)
+    (in_bom yes) (on_board yes) (dnp no)
     (property "Reference" "J2" (at 368.3 208.28 0)
       (effects (font (size 1.27 1.27)) (justify left) hide)
     )
-    (property "Value" "687110149022" (at 368.3 205.74 0)
+    (property "Value" "FPC 10pin 0.5mm pitch" (at 368.3 205.74 0)
       (effects (font (size 1.27 1.27)) (justify left) hide)
     )
@@
       (effects (font (size 1 1)))
     )
-    (pin "2")
+    (property "Link" "https://www.aliexpress.us/item/10000348360254.html" (at 368.3 205.74 0)
+      (effects (font (size 1.27 1.27)) hide)
+    )
+    (pin "2")

Commit message: doc
Parts:
- R4: Link (none) -> https://www.aliexpress.us/item/1005002364437129.html
Changed lines of the file:
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@@
+      (effects (font (size 1.27 1.27)) hide)
+    )
+    (property "Link" "https://www.aliexpress.us/item/1005002364437129.html" (at 201.93 233.68 0)
       (effects (font (size 1.27 1.27)) hide)
     )

Commit message: doc
Parts:
- D2: value LED BOTTOM -> 020 SMD Side View LED White 6000K; Link (none) -> https://www.aliexpress.us/item/32419907074.html; Role (none) -> Flashlight, Led bottom; now in the parts list
- S1, S2, S4: value TL3330AF130QG -> 2*4*3.5mm Micro SMD Tact Switch Side Button; Availability In Stock -> (none); Check_prices https://www.snapeda.com/parts/TL3330AF130QG/E-Switch/view-p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 -> (none); Link (none) -> https://www.aliexpress.us/item/32880903601.html; MANUFACTURER E-Switch -> (none); MAXIMUM_PACKAGE_HEIGHT 3.4 mm -> (none); MF E-Switch -> (none); MP TL3330AF130QG -> (none); PARTREV B -> (none); Package None -> (none); Price None -> (none); Purchase-URL https://www.snapeda.com/api/url_track_click_mouser/?unipart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 -> (none); SNAPEDA_PN TL3330AF130QG -> (none); STANDARD Manufacturer Recommendations -> (none); SnapEDA_Link https://www.snapeda.com/parts/TL3330AF130QG/E-Switch/view-p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 -> (none); now in the parts list
- S3: value TL3330AF130QG -> 2*4*3.5mm Micro SMD Tact Switch Side Button; Availability In Stock -> (none); Check_prices https://www.snapeda.com/parts/TL3330AF130QG/E-Switch/view-p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 -> (none); Link (none) -> https://www.aliexpress.us/item/32880903601.html; MANUFACTURER E-Switch -> (none); MAXIMUM_PACKAGE_HEIGHT 3.4 mm -> (none); MF E-Switch -> (none); MP TL3330AF130QG -> (none); PARTREV B -> (none); Package None -> (none); Price None -> (none); Purchase-URL https://www.snapeda.com/api/url_track_click_mouser/?unipart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 -> (none); SNAPEDA_PN TL3330AF130QG -> (none); STANDARD Manufacturer Recommendations -> (none); SnapEDA_Link https://www.snapeda.com/parts/TL3330AF130QG/E-Switch/view-p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 -> (none)
- U4: Link (none) -> https://www.analog.com/en/products/ds3231.html; Role (none) -> Handling Time

Commit message: 2024-04-02 Доповнено документацію 2024-04-03 Доповнено документацію
2024-04-02 Доповнено документацію
2024-04-03 Доповнено документацію
Parts:
- added TP39: RTCBAT, Project-Lib:TestPoint_Pad, symbol Project-Lib:TestPoint
- C1, C10, C14, C17, C18, C4, C5, C6, C7, C9: Link (none) -> https://www.aliexpress.us/item/1005006124283234.html
- C13: Link (none) -> https://www.aliexpress.us/item/1005006124283234.html; wewe haha4455 -> (none); now in the parts list
- C16: Link (none) -> https://www.aliexpress.us/item/1005004628006766.html
- C8: Link (none) -> https://www.aliexpress.us/item/1005006124283234.html; wewe haha4455 -> (none)
- M1, M2, M3: value ~ -> M1.2 screw mount get from DJI Mavic 3 CORE board; Link (none) -> https://www.aliexpress.com/i/1005005125674149.html (SMTSO-M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; now in the parts list
- R16: Link (none) -> https://www.aliexpress.us/item/1005002364437129.html
- S3: now in the parts list
- U2: value ~ -> ME6211 SOT23-5 3.3V; Datasheet2 (none) -> https://datasheetspdf.com/pdf-down/M/E/6/ME6211-Microne.pdf; Link (none) -> https://www.aliexpress.us/item/1005006036398325.html; now in the parts list
Connections:
- net at U4.14 (VBAT): now also TP39.1

Commit message: doc
Parts:
- added C19: 1uF, Project-Lib:C_0805_2012Metric, symbol Device:C
- added D7: US1D, Project-Lib:US1D, symbol Diode:US1D
- added Q2: 2N7002LT1G, Project-Lib:SOT95P240X111-3N, symbol Project-Lib:2N7002LT1G
- added R22: 1K, Project-Lib:R_0603_1608Metric, symbol Device:R
- added R23: R22, Project-Lib:R_0603_1608Metric, symbol Device:R
- added TP40: VIB+, Project-Lib:TestPoint_Pad, symbol Project-Lib:TestPoint
- added TP41: VIB-, Project-Lib:TestPoint_Pad, symbol Project-Lib:TestPoint
- added TP42: VIB, Project-Lib:TestPoint_Pad, symbol Project-Lib:TestPoint
- C13: value TBD -> 10pF
- J1: Availability Not in stock -> (none); Check_prices https://www.snapeda.com/parts/TYPE-C-31-M-12/HRO+Electronic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 -> (none); MAXIMUM_PACKAGE_HEIGHT 3.26 mm -> (none); MF HRO Electronics Co., Ltd. -> (none); MP TYPE-C-31-M-12 -> (none); PARTREV 2020.12.08 -> (none); Package Package -> (none); Price None -> (none); SNAPEDA_PN TYPE-C-31-M-12 -> (none); STANDARD Manufacturer Recommendations -> (none); now in the parts list
- R15: value TBD -> 0 ohm; now in the parts list
Connections:
- net GND: now also Q2.2, R22.2
- net VCC: now also R23.2
- net at U1.14 (GPIO9/ADC1_CH8): now also Q2.1, R22.1, TP42.1
- new net: C19.2, D7.1 (K), R23.1, TP40.1
- new net: C19.1, D7.2 (A), Q2.3, TP41.1
Other:
- note added: "VIBRATOR ZONE"
- moved on the sheet: C15, C16, C17, C18, D1, D2, D5, D6, L1, LS1, Q1, R1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

Commit message: docs
Parts:
- BT1: Role (none) -> Battery
- C1, C10, C4, C5, C6: Role (none) -> Voltage stabilizer capacitor for 3v3
- C13: Role (none) -> Capacitor to antenna
- C14: Role (none) -> Voltage stabilizer capacitor for EN pin
- C2, C3: Role (none) -> Capacitor for oscilator
- C7, C8: Role (none) -> Voltage stabilizer capacitor for VDD_SPI
- C9: Role (none) -> Voltage stabilizer capacitor for VBAT
- LS1: AVAILABILITY Unavailable -> (none); Availability In Stock -> (none); CUI_purchase_URL https://www.cuidevices.com/product/audio/buzzers/audio-tran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 -> (none); Check_prices https://www.snapeda.com/parts/CMT-7525S-SMT-TR/CUI+Devices/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 -> (none); DESCRIPTION 5 mm, 3 V, 75 dB, Surface Mount _SMT_, Magnetic Audio Trans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 -> (none); MF CUI Devices -> (none); MP CMT-7525S-SMT-TR -> (none); Manufacturer (none) -> CUI Devices; PACKAGE None -> (none); PRICE None -> (none); Package None -> (none); Price None -> (none); Purchase-URL https://www.snapeda.com/api/url_track_click_mouser/?unipart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 -> (none); Role (none) -> Buzzer to play sound; SnapEDA_Link https://www.snapeda.com/parts/CMT-7525S-SMT-TR/CUI+Devices/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 -> (none)
- M1, M2, M3: Role (none) -> Screw mount for back case
- Q1: value 2N7002LT1G -> 2N7002LT1G (SOT-23-3); Check_prices https://www.snapeda.com/parts/2N7002LT1G/Onsemi/view-part/?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 -> (none); Link (none) -> https://www.aliexpress.us/item/1005003909614901.html; Link2 (none) -> https://www.aliexpress.us/item/1005003079655220.html; MAXIMUM_PACKAGE_HEIGHT 1.11 mm -> (none); MF onsemi -> (none); MP 2N7002LT1G -> (none); PARTREV 4 -> (none); Package SOT-23-3 ON Semiconductor -> (none); Purchase-URL https://www.snapeda.com/api/url_track_click_mouser/?unipart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 -> (none); RS_Components_1032941_Purchase_URL https://www.snapeda.com/api/url_track_click/https%253A//uk.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 -> (none); RS_Components_5450012P_Purchase_URL https://www.snapeda.com/api/url_track_click/https%253A//uk.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 -> (none); RS_Components_5450012_Purchase_URL https://www.snapeda.com/api/url_track_click/https%253A//uk.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 -> (none); Role (none) -> Driving MOSFET for buzzer; STANDARD IPC 7351B -> (none); SnapEDA_Link https://www.snapeda.com/parts/2N7002LT1G/Onsemi/view-part/?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 -> (none); now in the parts list
- R1: Role (none) -> Pull-down for buzzer signal
- R11, R12: Role (none) -> Part of voltage divider for battery
- R13, R14: Role (none) -> Part of voltage divider for USB
- R15: Role (none) -> Resistor to antenna
- R16: Role (none) -> Pull-Up for ENABLE pin of ESP32
- R4: Role (none) -> Current-limiting ressitor for buzzer
- U1: Role (none) -> Main controller
- U2: Role (none) -> Step-down voltage converter
- Y1: Role (none) -> Frequency Oscilator

Commit message: schrmatic update
Parts:
- C11: Role (none) -> Capacitor for vbat
- C12: Role (none) -> Voltage stabilizing capacitor for usb
- D3: value LED STBY -> LED BLUE; Link (none) -> https://www.aliexpress.us/item/4000936781234.html; Role (none) -> LED STBY; now in the parts list
- D4: value LED CHARGE -> LED RED; Link (none) -> https://www.aliexpress.us/item/4000936781234.html; Role (none) -> LED CHARGE; now in the parts list
- J1: Link2 (none) -> https://www.snapeda.com/parts/TYPE-C-31-M-12/HRO+Electronic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; SnapEDA_Link https://www.snapeda.com/parts/TYPE-C-31-M-12/HRO+Electronic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 -> (none)
- JP1: now left out of the parts list
- R7: Role (none) -> Current-limit resistor for LED STBY
- R8: Role (none) -> Current limiting resistor for LED CHG
- R9: Role (none) -> Current setting resistor more 1K=1A, 10K=100mA
- U3: MF Texas Instruments -> (none); MP TP4056 -> (none); Manufacturer (none) -> Texas Instruments; Role (none) -> Battery charger; now in the parts list
Changed lines of the file:
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@@
   )
   (rectangle (start 20.32 119.38) (end 119.38 176.53)
-    (stroke (width 0) (type dash) (color 132 132 132 1))
-    (fill (type none))
+    (stroke (width 0) (type dash) (color 0 194 194 1))
+    (fill (type color) (color 255 255 255 1))
   )
   (rectangle (start 120.65 210.82) (end 161.29 254)
@@
   )
   (symbol (lib_id "Project-Lib:TP4056") (at 64.77 137.16 0) (unit 1)
-    (in_bom no) (on_board yes) (dnp no) (fields_autoplaced)
+    (in_bom yes) (on_board yes) (dnp no) (fields_autoplaced)
     (property "Reference" "U3" (at 64.77 121.92 0)
       (effects (font (size 1.27 1.27)))
@@
       (effects (font (size 1.27 1.27)) hide)
     )
-    (property "MF" "Texas Instruments" (at 64.77 116.84 0)
-      (effects (font (size 1.27 1.27)) (justify bottom) hide)
-    )
-    (property "MP" "TP4056" (at 67.31 119.38 0)
+    (property "Manufacturer" "Texas Instruments" (at 64.77 116.84 0)
       (effects (font (size 1.27 1.27)) (justify bottom) hide)
     )
@@
       (effects (font (size 1.27 1.27)) hide)
     )
+    (property "Role" "Battery charger" (at 64.77 137.16 0)
+      (effects (font (size 1.27 1.27)) hide)
+    )
     (pin "5")
     (pin "6")
@@
       (effects (font (size 1.27 1.27)) hide)
     )
+    (property "Role" "Voltage stabilizing capacitor for usb" (at 48.26 157.48 90)
+      (effects (font (size 1.27 1.27)) hide)
+    )
     (pin "2")
     (pin "1")
@@
   )
   (symbol (lib_id "Jumper:Jumper_2_Open") (at 100.33 171.45 180) (unit 1)
-    (in_bom yes) (on_board yes) (dnp no) (fields_autoplaced)
-    (property "Reference" "JP1" (at 100.33 166.37 0)
+    (in_bom no) (on_board yes) (dnp no) (fields_autoplaced)
+    (property "Reference" "JP1" (at 100.33 167.64 0)
       (effects (font (size 1.27 1.27)))
     )
     (property "Value" "Connect this to directly power VCC from USB" (at 100.33 168.91 0)
-      (effects (font (size 1.27 1.27)))
+      (effects (font (size 0.67 0.67)))
     )
     (property "Footprint" "Project-Lib:SolderJumper-2_P1.3mm_Open_Pad1.0x1.5mm" (at 100.33 171.45 0)
@@
       (effects (font (size 1.27 1.27)) hide)
     )
+    (property "Role" "Capacitor for vbat" (at 77.47 152.4 90)
+      (effects (font (size 1.27 1.27)) hide)
+    )
     (pin "2")
     (pin "1")
@@
   )
   (symbol (lib_id "Device:LED") (at 91.44 157.48 270) (unit 1)
-    (in_bom no) (on_board yes) (dnp no) (fields_autoplaced)
+    (in_bom yes) (on_board yes) (dnp no) (fields_autoplaced)
     (property "Reference" "D4" (at 93.98 154.6225 90)
       (effects (font (size 1.27 1.27)) (justify left))
     )
-    (property "Value" "LED CHARGE" (at 93.98 157.1625 90)
+    (property "Value" "LED RED" (at 93.98 157.1625 90)
       (effects (font (size 1.27 1.27)) (justify left))
     )
@@
       (effects (font (size 1.27 1.27)) hide)
     )
+    (property "Role" "LED CHARGE" (at 91.44 157.48 90)
+      (effects (font (size 1.27 1.27)) hide)
+    )
+    (property "Link" "https://www.aliexpress.us/item/4000936781234.html" (at 91.44 157.48 90)
+      (effects (font (size 1.27 1.27)) hide)
+    )
     (pin "2")
     (pin "1")
@@
   )
   (symbol (lib_id "Device:LED") (at 92.71 144.78 270) (unit 1)
-    (in_bom no) (on_board yes) (dnp no) (fields_autoplaced)
+    (in_bom yes) (on_board yes) (dnp no) (fields_autoplaced)
     (property "Reference" "D3" (at 95.25 141.9225 90)
       (effects (font (size 1.27 1.27)) (justify left))
     )
-    (property "Value" "LED STBY" (at 95.25 144.4625 90)
+    (property "Value" "LED BLUE" (at 95.25 144.4625 90)
       (effects (font (size 1.27 1.27)) (justify left))
     )
@@
       (effects (font (size 1.27 1.27)) hide)
     )
+    (property "Link" "https://www.aliexpress.us/item/4000936781234.html" (at 92.71 144.78 90)
+      (effects (font (size 1.27 1.27)) hide)
+    )
+    (property "Role" "LED STBY" (at 92.71 144.78 90)
+      (effects (font (size 1.27 1.27)) hide)
+    )
     (pin "2")
     (pin "1")
@@
       (effects (font (size 1.27 1.27)) hide)
     )
+    (property "Role" "Current setting resistor more 1K=1A, 10K=100mA" (at 26.67 140.97 0)
+      (effects (font (size 1.27 1.27)) hide)
+    )
     (pin "1")
     (pin "2")
@@
       (effects (font (size 1.27 1.27)) hide)
     )
-    (property "SnapEDA_Link" "https://www.snapeda.com/parts/TYPE-C-31-M-12/HRO+Electronics+Co.%252C+Ltd./view-part/?ref=snap" (at 355.6 30.48 0)
+    (property "Link2" "https://www.snapeda.com/parts/TYPE-C-31-M-12/HRO+Electronics+Co.%252C+Ltd./view-part/?ref=snap" (at 355.6 30.48 0)
       (effects (font (size 1.27 1.27)) (justify bottom) hide)
     )
@@
     )
   )
-  (symbol (lib_id "Project-Lib:2N7002LT1G") (at 130.81 234.95 0) (unit 1)
+  (symbol (lib_name "2N7002LT1G_1") (lib_id "Project-Lib:2N7002LT1G") (at 130.81 234.95 0) (unit 1)
     (in_bom yes) (on_board yes) (dnp no)
     (property "Reference" "Q1" (at 135.89 234.95 0)
@@
       (effects (font (size 1.27 1.27)) hide)
     )
+    (property "Role" "Current limiting resistor for LED CHG" (at 109.22 158.75 0)
+      (effects (font (size 1.27 1.27)) hide)
+    )
     (pin "1")
     (pin "2")
@@
       (effects (font (size 1.27 1.27)) hide)
     )
+    (property "Role" "Current-limit resistor for LED STBY" (at 107.95 146.05 0)
+      (effects (font (size 1.27 1.27)) hide)
+    )

Commit message: 2024-04-17 Трохи оновлено модель 2024-04-17 Додано файли для гравіювання передньої панелі 2024-04-17 Доповнено схему
2024-04-17 Трохи оновлено модель
2024-04-17 Додано файли для гравіювання передньої панелі
2024-04-17 Доповнено схему
Parts:
- C11, C12, C15, C2, C3: Link (none) -> https://www.aliexpress.us/item/1005006124283234.html
- C16: Model Capacitor SMD 1206 10NF X7R 200V -> (none); Role (none) -> Complementary component for EL driver chip
- D6: Link (none) -> https://www.aliexpress.us/item/1005005254835443.html; Role (none) -> Complementary part for EL driver chip
- D7: Link (none) -> https://www.aliexpress.us/item/1005005254835443.html
- J1: MANUFACTURER HRO Electronics Co., Ltd. -> (none); Manufacturer (none) -> HRO Electronics Co., Ltd.
- J2: Availability In Stock -> (none); Check_prices https://www.snapeda.com/parts/687110149022/Wurth+Electronic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 -> (none); MF Wurth Electronics -> (none); MP 687110149022 -> (none); Package None -> (none); Price None -> (none); Role LCD -> LCD Connector; SnapEDA_Link https://www.snapeda.com/parts/687110149022/Wurth+Electronic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 -> (none); pin1 desc LCD SCL -> (none); pin10 desc LCD GNDA -> (none); pin2 desc LCD SDA -> (none); pin3 desc LCD CS -> (none); pin4 desc LCD EXTCOMIN -> (none); pin5 desc LCD ON OFF -> (none); pin6 desc LCD VDDA -> (none); pin7 desc LCD VDD -> (none); pin8 desc LCD EXTMODE -> (none); pin9 desc LCD GND -> (none)
- L1: Link (none) -> https://www.aliexpress.us/item/32981310345.html; Role (none) -> Complementary part for EL driver chip
- Q1: MANUFACTURER ON Semiconductor -> (none); Manufacturer (none) -> ON Semiconductor
- U2: Datasheet2 https://datasheetspdf.com/pdf-down/M/E/6/ME6211-Microne.pdf -> (none)
- U4: Availability In Stock -> (none); Check_prices https://www.snapeda.com/parts/DS3231S/Analog+Devices/view-p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 -> (none); MF Analog Devices -> (none); MP DS3231S -> (none); Manufacturer (none) -> Analog Devices; Package SOIC-16 Maxim -> (none); Price None -> (none); Purchase-URL https://www.snapeda.com/api/url_track_click_mouser/?unipart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 -> (none); SnapEDA_Link https://www.snapeda.com/parts/DS3231S/Analog+Devices/view-p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 -> (none)
- Y1: Manufacturer (none) -> Murata Electronics; Package 3225 smd -> (none)
