File: Board/_DRM_Watch_v3/DRM_Watch_V3.kicad_pcb (KiCad board)
At the start: 2 copper layers, 62.7 x 44.4 mm, 107 parts, among them J1 TYPE-C-31-M-12, J2 687110149022, Q1 2N7002LT1G, U1 ESP32-S2, U3 TP4056, U4 DS3231S, Y1 XRCGB48M000F0Z00R0

Commit message: doc
Parts:
- added C19: 1uF, Project-Lib:C_0805_2012Metric, F.Cu at (146.1, 56.0)
- added D7: US1D, Project-Lib:US1D, F.Cu at (143.9, 47.8)
- added Q2: 2N7002LT1G, Project-Lib:SOT95P240X111-3N, F.Cu at (146.3, 52.3)
- added R22: 1K, Project-Lib:R_0603_1608Metric, F.Cu at (141.8, 51.3)
- added R23: R22, Project-Lib:R_0603_1608Metric, F.Cu at (141.8, 53.8)
- added TP39: RTCBAT, Project-Lib:TestPoint_Pad, F.Cu at (138.0, 59.5)
- added TP40: VIB+, Project-Lib:TestPoint_Pad, F.Cu at (138.0, 62.8)
- added TP41: VIB-, Project-Lib:TestPoint_Pad, F.Cu at (138.0, 66.0)
- added TP42: VIB, Project-Lib:TestPoint_Pad, F.Cu at (149.5, 47.1)
- C13: value TBD -> 10pF
- D2: value LED BOTTOM -> 020 SMD Side View LED White 6000K
- J2: value 687110149022 -> FPC 10pin 0.5mm pitch
- M1, M2, M3: value ~ -> M1.2 screw mount get from DJI Mavic 3 CORE board
- R15: value TBD -> 0 ohm
- S1, S2, S3, S4: value TL3330AF130QG -> 2*4*3.5mm Micro SMD Tact Switch Side Button
- U2: value ~ -> ME6211 SOT23-5 3.3V
- U5: value ~ -> Microchip HV857
- Y1: value XRCGB48M000F0Z00R0 -> 3225 4PIN 40Mhz 3.2*2.5mm Passive SMD Quartz Resonator Crystal
Connections:
- U1 pad 14: unconnected-(U1-GPIO9/ADC1_CH8-Pad14) -> Net-(U1-GPIO9/ADC1_CH8)
- U4 pad 14: unconnected-(U4-VBAT-Pad14) -> Net-(U4-VBAT)

Commit message: 2024-04-18 Оновлено схему 2024-04-18 Оновлено Плату 2024-04-18 Оновлено Production файли для плати rev4
2024-04-18 Оновлено схему
2024-04-18 Оновлено Плату
2024-04-18 Оновлено Production файли для плати rev4
Parts:
- D1: value LED TOP -> LED RED
- D3: value LED STBY -> LED BLUE
- D4: value LED CHARGE -> LED RED
- D5: value LED STATUS -> LED BLUE
- Q1, Q2: value 2N7002LT1G -> 2N7002LT1G (SOT-23-3)
- TP36, TP8: moved to F.Cu
- TP42: moved to B.Cu
- moved D7 41.1 mm to (118.9, 80.4), turned to -90 degrees
- moved TP8 40.1 mm to (113.8, 72.5), turned to 0 degrees
- moved TP42 38.6 mm to (120.5, 72.5)
- moved C19 36.0 mm to (122.4, 83.1)
- moved Q2 35.6 mm to (118.9, 74.9), turned to -90 degrees
- moved R23 33.6 mm to (125.6, 83.2)
- moved TP39 29.6 mm to (112.3, 74.2)
- moved R22 29.3 mm to (122.3, 73.1)
- moved TP41 26.2 mm to (120.0, 85.0)
- moved TP40 25.8 mm to (125.0, 85.0)
- moved Q1 18.9 mm to (113.1, 59.1), turned to 180 degrees
- moved TP22 17.2 mm to (112.5, 58.5)
- moved TP28 11.0 mm to (110.5, 72.5)
- moved C14 10.9 mm to (125.4, 74.6), turned to 180 degrees
- moved R16 10.6 mm to (122.3, 74.6)
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Routing:
- net VCC: track 126.8 -> 180.4 mm, vias 3 -> 5
- net Net-(U1-GPIO9/ADC1_CH8): track 0.00 -> 43.6 mm, vias 0 -> 3
- net GND: track 31.2 -> 54.1 mm, vias 38 -> 39
- net Net-(D7-A): track 0.00 -> 12.8 mm
- net Net-(U4-VBAT): track 0.00 -> 11.6 mm
- net Net-(U1-GPIO12/ADC2_CH1): track 32.5 -> 21.9 mm
- net Net-(D7-K): track 0.00 -> 9.98 mm
- net +3V3: track 167.8 -> 175.5 mm, vias 4 -> 6
- net Net-(U1-CHIP_PU/RESET): track 62.5 -> 56.3 mm, vias 3 -> 2
- net Net-(LS1-PadN): track 6.95 -> 13.1 mm
- net Net-(J1-DN1): track 16.1 -> 21.4 mm
- net Net-(J1-DP1): track 13.8 -> 18.9 mm
- net Net-(U1-GPIO14/ADC2_CH3): track 7.55 -> 5.57 mm
- net Net-(U1-GPIO38): track 64.7 -> 63.3 mm
- net Net-(J1-CC2): track 11.7 -> 10.4 mm
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Other:
- board text added: "Rev.4 (2024-04-18)"
- board text removed: "Rev.3 (2024-03-02)"
